File: AVRProgrammer.sch (KiCad schematic (older format))
At the start: 7 parts, among them IC1 ATMEGA32-P, J1 AVR-ISP-6

Commit message: modified:   AVRProgrammer.brd 	modified:   AVRProgrammer.cmp 	deleted:    AVRProgrammer.drl 	modified:   AVRProgrammer.net 	modified:   AVRProgrammer.pro 	modified:   AVRProgrammer.sch 	Gerber/
Parts:
- removed IC1: ATMEGA32-P, DIL40, symbol ATMEGA32-P
- removed J1: AVR-ISP-6, AVR-ISP-6, symbol AVR-ISP-6
- added C2, C3: 27pf, symbol C
- added CON1: AVR-ISP-6, AVR-ISP-6, symbol AVR-ISP-6
- added P1: 40PIN_component, symbol 40PIN_component
- added P2: jumper, symbol CONN_2
- added X1: OSCILLATOR, symbol OSCILLATOR
- R2: value R -> 470
Connections:
- net labels added: clk1, clk2, miso, mosi, rst, sck
Other:
- moved on the sheet: C1, D1, D2, R1, R2

Commit message: modified:   AVRProgrammer.brd 	modified:   AVRProgrammer.cmp 	modified:   AVRProgrammer.net 	modified:   AVRProgrammer.sch 	modified:   Gerber/AVRProgrammer-Back.gbl 	modified:   Gerber/AVRProgrammer-Front.gtl 	modified:   Gerber/AVRProgrammer-Mask_Back.gbs 	modified:   Gerber/AVRProgrammer-Mask_Front.gts 	modified:   Gerber/AVRProgrammer-PCB_Edges.gbr 	modified:   Gerber/AVRProgrammer-SilkS_Back.gbo 	modified:   Gerber/AVRProgrammer-SilkS_Front.gto 	modified:   Gerber/AVRProgrammer-drl.rpt 	modified:   Gerber/AVRProgrammer.drl
Parts:
- added D3: LED, symbol LED
- added R3: 220, symbol R
- added SW1: SPST, symbol SPST
- R1: value 180 -> 220
- R2: value 470 -> 220
Connections:
- net labels added: led_test
- wire segments 44 -> 50
Other:
- note added: "pd5 - ATMEGA328\npb4 - ATTiny85"
Changed lines of the file:
@@
-EESchema Schematic File Version 2  date Fri 30 Mar 2012 10:02:04 PM EDT
+EESchema Schematic File Version 2  date Sat 16 Jun 2012 05:29:30 AM EDT
 LIBS:power
 LIBS:device
@@
 Sheet 1 1
 Title ""
-Date "31 mar 2012"
+Date "16 jun 2012"
 Rev ""
 Comp ""
@@
 $EndDescr
 Wire Wire Line
-	4500 4000 4950 4000
+	1550 3350 2050 3350
+Wire Wire Line
+	1550 3150 2050 3150
+Wire Wire Line
+	9600 3100 9600 2850
+Wire Wire Line
+	2950 1150 2950 1550
+Connection ~ 4950 3900
+Wire Wire Line
+	4950 3900 4950 4000
+Wire Wire Line
+	5400 4000 5050 4000
+Wire Wire Line
+	5050 4000 5050 4200
+Wire Wire Line
+	5050 4200 5000 4200
+Connection ~ 7350 3150
+Wire Wire Line
+	7350 2800 7350 3150
+Wire Wire Line
+	7900 3150 8100 3150
+Wire Wire Line
+	8100 3150 8100 4100
+Wire Wire Line
+	7200 3750 7200 3800
+Wire Wire Line
+	7200 3800 7500 3800
+Wire Wire Line
+	2350 3350 2850 3350
+Wire Wire Line
+	4900 3900 5400 3900
+Wire Wire Line
+	6350 4200 6200 4200
+Connection ~ 6250 3800
+Wire Wire Line
+	6250 3800 6250 3900
+Wire Wire Line
+	6250 3900 6200 3900
+Wire Wire Line
+	6200 3700 6500 3700
+Wire Wire Line
+	6500 3700 6500 3800
+Wire Wire Line
+	5050 3700 5400 3700
+Wire Wire Line
+	3050 3950 3050 3250
+Wire Wire Line
+	3050 4450 3050 4650
+Wire Wire Line
+	3450 3750 3450 3950
+Wire Wire Line
+	5450 1850 5450 2050
+Wire Wire Line
+	2850 3350 2850 3650
+Wire Wire Line
+	5450 2450 5450 2650
+Wire Wire Line
+	3450 4450 3450 4650
+Wire Wire Line
+	3450 5050 3450 5350
+Wire Wire Line
+	3050 5050 3050 5350
+Connection ~ 3050 3250
+Wire Wire Line
+	5050 3100 5400 3100
+Wire Wire Line
+	6200 3800 6300 3800
+Wire Wire Line
+	6350 4100 6200 4100
+Wire Wire Line
+	6350 4000 6200 4000
+Wire Wire Line
+	5000 3800 5400 3800
+Wire Wire Line
+	3300 3250 2350 3250
+Wire Wire Line
+	5400 4200 5200 4200
+Wire Wire Line
+	5200 4200 5200 4250
+Wire Wire Line
+	7200 3150 7500 3150
+Wire Wire Line
+	7900 3800 8100 3800
+Connection ~ 8100 3800
+Wire Wire Line
+	7350 4300 7350 3800
+Connection ~ 7350 3800
 Wire Wire Line
 	4600 4200 4500 4200
-Connection ~ 7350 3800
-Wire Wire Line
-	7350 4300 7350 3800
-Connection ~ 8100 3800
-Wire Wire Line
-	7900 3800 8100 3800
-Wire Wire Line
-	7500 3150 7200 3150
-Wire Wire Line
-	5200 4250 5200 4200
-Wire Wire Line
-	5200 4200 5400 4200
-Wire Wire Line
-	2350 3250 3300 3250
-Wire Wire Line
-	2050 3350 1850 3350
-Wire Wire Line
-	2050 3150 1850 3150
-Wire Wire Line
-	5000 3800 5400 3800
-Wire Wire Line
-	6350 4000 6200 4000
-Wire Wire Line
-	6350 4100 6200 4100
-Wire Wire Line
-	6300 3800 6200 3800
-Wire Wire Line
-	5050 3100 5400 3100
-Connection ~ 3050 3250
-Wire Wire Line
-	3050 5050 3050 5350
-Wire Wire Line
-	3450 5050 3450 5350
-Wire Wire Line
-	3450 4450 3450 4650
-Wire Wire Line
-	5450 2450 5450 2650
-Wire Wire Line
-	2900 2750 2900 3150
-Wire Wire Line
-	2850 3650 2850 3350
-Wire Wire Line
-	5450 1850 5450 2050
-Wire Wire Line
-	3450 3750 3450 3950
-Wire Wire Line
-	3050 4450 3050 4650
-Wire Wire Line
-	3050 3250 3050 3950
-Wire Wire Line
-	5050 3700 5400 3700
-Wire Wire Line
-	6500 3800 6500 3700
-Wire Wire Line
-	6500 3700 6200 3700
-Wire Wire Line
-	6200 3900 6250 3900
-Wire Wire Line
-	6250 3900 6250 3800
-Connection ~ 6250 3800
-Wire Wire Line
-	6350 4200 6200 4200
-Wire Wire Line
-	5400 3900 4900 3900
-Wire Wire Line
-	2050 3250 1850 3250
-Wire Wire Line
-	2850 3350 2350 3350
-Wire Wire Line
-	2900 3150 2350 3150
-Wire Wire Line
-	7500 3800 7200 3800
-Wire Wire Line
-	7200 3800 7200 3750
-Wire Wire Line
-	8100 4100 8100 3150
-Wire Wire Line
-	8100 3150 7900 3150
-Wire Wire Line
-	7350 2800 7350 3150
-Connection ~ 7350 3150
-Wire Wire Line
-	5000 4200 5050 4200
-Wire Wire Line
-	5050 4200 5050 4000
-Wire Wire Line
-	5050 4000 5400 4000
-Wire Wire Line
-	4950 4000 4950 3900
-Connection ~ 4950 3900
+Wire Wire Line
+	4950 4000 4500 4000
+Wire Wire Line
+	2950 2550 2950 3150
+Wire Wire Line
+	2950 3150 2350 3150
+Wire Wire Line
+	9600 2250 9600 2450
+Wire Wire Line
+	9600 1550 9600 1750
+Wire Wire Line
+	5100 4500 5100 4100
+Wire Wire Line
+	5100 4100 5400 4100
+Wire Wire Line
+	1550 3250 2050 3250
+Text Label 5100 4500 3    60   ~ 0
+led_test
+Text Notes 9800 3150 0    60   ~ 0
+pd5 - ATMEGA328\npb4 - ATTiny85
+Text Label 9600 3100 3    60   ~ 0
+led_test
+$Comp
+L LED D3
+U 1 1 4FDBF9AD
+P 9600 2650
+F 0 "D3" H 9600 2750 50  0000 C CNN
+F 1 "LED" H 9600 2550 50  0000 C CNN
+	1    9600 2650
+	0    1    1    0
+$EndComp
+$Comp
+L R R3
+U 1 1 4FDBF9A7
+P 9600 2000
+F 0 "R3" V 9680 2000 50  0000 C CNN
+F 1 "220" V 9600 2000 50  0000 C CNN
+	1    9600 2000
+	1    0    0    -1
+$EndComp
+$Comp
+L VCC #PWR01
+U 1 1 4FDBF9A1
+P 9600 1550
+F 0 "#PWR01" H 9600 1650 30  0001 C CNN
+F 1 "VCC" H 9600 1650 30  0000 C CNN
+	1    9600 1550
+	1    0    0    -1
+$EndComp
+$Comp
+L SPST SW1
+U 1 1 4FDBF498
+P 2950 2050
+F 0 "SW1" H 2950 2150 70  0000 C CNN
+F 1 "SPST" H 2950 1950 70  0000 C CNN
+	1    2950 2050
+	0    -1   -1   0
+$EndComp
 $Comp
 L 40PIN_component P1
@@
 clk1
 $Comp
-L GND #PWR01
+L GND #PWR02
 U 1 1 4F7661EC
 P 8100 4100
-F 0 "#PWR01" H 8100 4100 30  0001 C CNN
+F 0 "#PWR02" H 8100 4100 30  0001 C CNN
 F 1 "GND" H 8100 4030 30  0001 C CNN
 	1    8100 4100
@@
 $EndComp
 $Comp
-L GND #PWR02
+L GND #PWR03
 U 1 1 4F67E47F
 P 5200 4250
-F 0 "#PWR02" H 5200 4250 30  0001 C CNN
+F 0 "#PWR03" H 5200 4250 30  0001 C CNN
 F 1 "GND" H 5200 4180 30  0001 C CNN
 	1    5200 4250
@@
 miso
 $Comp
-L VCC #PWR03
+L VCC #PWR04
 U 1 1 4F67E32A
 P 6300 3800
-F 0 "#PWR03" H 6300 3900 30  0001 C CNN
+F 0 "#PWR04" H 6300 3900 30  0001 C CNN
 F 1 "VCC" H 6300 3900 30  0000 C CNN
 	1    6300 3800
@@
 $EndComp
 $Comp
-L GND #PWR04
+L GND #PWR05
 U 1 1 4F67E300
 P 6500 3800
-F 0 "#PWR04" H 6500 3800 30  0001 C CNN
+F 0 "#PWR05" H 6500 3800 30  0001 C CNN
 F 1 "GND" H 6500 3730 30  0001 C CNN
 	1    6500 3800
@@
 $EndComp
 $Comp
-L GND #PWR05
+L GND #PWR06
 U 1 1 4F67E2D1
 P 5000 3800
-F 0 "#PWR05" H 5000 3800 30  0001 C CNN
+F 0 "#PWR06" H 5000 3800 30  0001 C CNN
 F 1 "GND" H 5000 3730 30  0001 C CNN
 	1    5000 3800
@@
 $EndComp
 $Comp
-L VCC #PWR06
+L VCC #PWR07
 U 1 1 4F67E297
 P 5050 3700
-F 0 "#PWR06" H 5050 3800 30  0001 C CNN
+F 0 "#PWR07" H 5050 3800 30  0001 C CNN
 F 1 "VCC" H 5050 3800 30  0000 C CNN
 	1    5050 3700
@@
 Text Label 5050 3100 2    60   ~ 0
 rst
-Text Label 1850 3350 2    60   ~ 0
+Text Label 1550 3350 2    60   ~ 0
 rst
-Text Label 1850 3250 2    60   ~ 0
+Text Label 1550 3250 2    60   ~ 0
 sck
-Text Label 1850 3150 2    60   ~ 0
+Text Label 1550 3150 2    60   ~ 0
 miso
 Text Label 3300 3250 0    60   ~ 0
@@
 P 3050 4200
 F 0 "R1" V 3130 4200 50  0000 C CNN
-F 1 "180" V 3050 4200 50  0000 C CNN
+F 1 "220" V 3050 4200 50  0000 C CNN
 	1    3050 4200
 	1    0    0    -1
@@
 $EndComp
 $Comp
-L GND #PWR07
+L GND #PWR08
 U 1 1 4E9A1E82
 P 3050 5350
-F 0 "#PWR07" H 3050 5350 30  0001 C CNN
+F 0 "#PWR08" H 3050 5350 30  0001 C CNN
 F 1 "GND" H 3050 5280 30  0001 C CNN
 	1    3050 5350
@@
 $EndComp
 $Comp
-L GND #PWR08
+L GND #PWR09
 U 1 1 4E9A1E50
 P 3450 5350
-F 0 "#PWR08" H 3450 5350 30  0001 C CNN
+F 0 "#PWR09" H 3450 5350 30  0001 C CNN
 F 1 "GND" H 3450 5280 30  0001 C CNN
 	1    3450 5350
@@
 $EndComp
 $Comp
-L VCC #PWR09
+L VCC #PWR010
 U 1 1 4E9A1E4E
 P 3450 3750
-F 0 "#PWR09" H 3450 3850 30  0001 C CNN
+F 0 "#PWR010" H 3450 3850 30  0001 C CNN
 F 1 "VCC" H 3450 3850 30  0000 C CNN
 	1    3450 3750
@@
 P 3450 4200
 F 0 "R2" V 3530 4200 50  0000 C CNN
-F 1 "470" V 3450 4200 50  0000 C CNN
+F 1 "220" V 3450 4200 50  0000 C CNN
 	1    3450 4200
 	1    0    0    -1
@@
 $EndComp
 $Comp
-L GND #PWR010
+L GND #PWR011
 U 1 1 4E9A1E26
 P 5450 2650
-F 0 "#PWR010" H 5450 2650 30  0001 C CNN
+F 0 "#PWR011" H 5450 2650 30  0001 C CNN
 F 1 "GND" H 5450 2580 30  0001 C CNN
 	1    5450 2650
@@
 $EndComp
 $Comp
-L VCC #PWR011
+L VCC #PWR012
 U 1 1 4E9A1E22
 P 5450 1850
-F 0 "#PWR011" H 5450 1950 30  0001 C CNN
+F 0 "#PWR012" H 5450 1950 30  0001 C CNN
 F 1 "VCC" H 5450 1950 30  0000 C CNN
 	1    5450 1850
@@
 $EndComp
 $Comp
-L VCC #PWR012
+L VCC #PWR013
 U 1 1 4E9A1C69
-P 2900 2750
-F 0 "#PWR012" H 2900 2850 30  0001 C CNN
-F 1 "VCC" H 2900 2850 30  0000 C CNN
-	1    2900 2750
-	1    0    0    -1
-$EndComp
-$Comp
-L GND #PWR013
+P 2950 1150
+F 0 "#PWR013" H 2950 1250 30  0001 C CNN
+F 1 "VCC" H 2950 1250 30  0000 C CNN
+	1    2950 1150
+	1    0    0    -1
+$EndComp
+$Comp
+L GND #PWR014
 U 1 1 4E9A1C5F
 P 2850 3650
-F 0 "#PWR013" H 2850 3650 30  0001 C CNN
+F 0 "#PWR014" H 2850 3650 30  0001 C CNN
 F 1 "GND" H 2850 3580 30  0001 C CNN
 	1    2850 3650
